Commit message: urdf fix

File: ros2_ws/src/bot_ws/src/startup_cpp/urdf/gptpet.xacro (robot description, xacro)
@@ -95,3 +95,130 @@
       </material>
     </visual>
-  </link>
+    <collision>
+      <origin xyz="0 0 0" rpy="0 0 0"/>
+      <geometry>
+        <box size="0.12 0.05 0.07"/>
+      </geometry>
+    </collision>
+    <inertial>
+      <mass value="0.5"/>
+      <inertia ixx="0.002" ixy="0" ixz="0" iyy="0.002" iyz="0" izz="0.002"/>
+    </inertial>
+  </link>
+  <joint name="laser_joint" type="fixed">
+    <parent link="base_link"/>
+    <child  link="base_laser_link"/>
+    <origin xyz="0 0.08 ${body_height/2 + kinect_height/2 + kinect_offset}" rpy="0 0 0"/>
+  </joint>
+  <!-- ========= JOINTS ========= -->
+  <xacro:macro name="wheel_origin" params="x_reflect y_reflect">
+    <parent link="base_link"/>
+    <origin xyz="${x_reflect * (body_width/2 + wheel_length/2 + wheel_offset_side)} ${y_reflect * wheel_separation_length/2} ${-body_height/2 -wheel_separation_down}" rpy="0 0 0"/>
+    <axis  xyz="0 0 1"/>
+  </xacro:macro>
+  <joint name="velocity_left_1_joint" type="continuous">
+    <child link="wheel_left_1_link"/>
+    <xacro:wheel_origin x_reflect="1" y_reflect="1" />
+  </joint>
+  <joint name="velocity_left_2_joint" type="continuous">
+    <child link="wheel_left_2_link"/>
+    <xacro:wheel_origin x_reflect="-1" y_reflect="1" />
+  </joint>
+  <joint name="velocity_right_1_joint" type="continuous">
+    <child  link="wheel_right_1_link"/>
+    <xacro:wheel_origin x_reflect="1" y_reflect="-1" />
+  </joint>
+  <joint name="velocity_right_2_joint" type="continuous">
+    <child link="wheel_right_2_link"/>
+    <xacro:wheel_origin x_reflect="-1" y_reflect="-1" />
+  </joint>
+  <!-- ========= TRANSMISSIONS ========= -->
+  <transmission name="trans_vel_left_1">
+    <type>transmission_interface/SimpleTransmission</type>
+    <joint name="velocity_left_1_joint">
+      <hardwareInterface>velocity</hardwareInterface>
+    </joint>
+    <actuator name="motor_left_1">
+      <hardwareInterface>velocity</hardwareInterface>
+      <mechanicalReduction>1</mechanicalReduction>
+    </actuator>
+  </transmission>
+  <transmission name="trans_vel_left_2">
+    <type>transmission_interface/SimpleTransmission</type>
+    <joint name="velocity_left_2_joint">
+      <hardwareInterface>velocity</hardwareInterface>
+    </joint>
+    <actuator name="motor_left_2">
+      <hardwareInterface>velocity</hardwareInterface>
+      <mechanicalReduction>1</mechanicalReduction>
+    </actuator>
+  </transmission>
+  <transmission name="trans_vel_right_1">
+    <type>transmission_interface/SimpleTransmission</type>
+    <joint name="velocity_right_1_joint">
+      <hardwareInterface>velocity</hardwareInterface>
+    </joint>
+    <actuator name="motor_right_1">
+      <hardwareInterface>velocity</hardwareInterface>
+      <mechanicalReduction>1</mechanicalReduction>
+    </actuator>
+  </transmission>
+  <transmission name="trans_vel_right_2">
+    <type>transmission_interface/SimpleTransmission</type>
+    <joint name="velocity_right_2_joint">
+      <hardwareInterface>velocity</hardwareInterface>
+    </joint>
+    <actuator name="motor_right_2">
+      <hardwareInterface>velocity</hardwareInterface>
+      <mechanicalReduction>1</mechanicalReduction>
+    </actuator>
+  </transmission>
+  <!-- ========= Cameras ========= -->
+  <link name="camera_link"/>
+  <joint name="camera_link_joint" type="fixed">
+    <parent link="base_laser_link"/>
+    <child link="camera_link"/>
+    <origin xyz="0 0 0" rpy="0 0 0"/>
+  </joint>
+  <link name="camera_depth_frame"/>
+  <joint name="camera_depth_joint" type="fixed">
+    <parent link="camera_link"/>
+    <child link="camera_depth_frame"/>
+    <origin xyz="0 0 0" rpy="0 0 0"/>
+  </joint>
+  <link name="camera_rgb_frame"/>
+  <joint name="camera_rgb_joint" type="fixed">
+    <parent link="camera_link"/>
+    <child link="camera_rgb_frame"/>
+    <origin xyz="0 0 0" rpy="0 0 0"/>
+  </joint>
+  <link name="camera_rgb_optical_frame"/>
+  <joint name="camera_rgb_optical_joint" type="fixed">
+    <parent link="camera_rgb_frame"/>
+    <child link="camera_rgb_optical_frame"/>
+    <origin xyz="0 0 0" rpy="-1.5708 0 -1.5708"/>
+  </joint>
+  <!-- ========= ROS2_CONTROL PLUGIN ========= -->
+  <ros2_control name="gptpet" type="system">
+    <hardware>
+      <!-- Reference the exported plugin name -->
+      <plugin>gptpet_hardware/GptpetHardwareInterface</plugin>
+    </hardware>
+    <joint name="velocity_left_1_joint">
+      <command_interface name="velocity"/>
+      <state_interface name="velocity"/>
+    </joint>
+    <joint name="velocity_left_2_joint">
+      <command_interface name="velocity"/>
+      <state_interface name="velocity"/>
+    </joint>
+    <joint name="velocity_right_1_joint">
+      <command_interface name="velocity"/>
+      <state_interface name="velocity"/>
+    </joint>
+    <joint name="velocity_right_2_joint">
+      <command_interface name="velocity"/>
+      <state_interface name="velocity"/>
+    </joint>
+  </ros2_control>
+</robot>
